File: z2m_partner.kicad_pcb (KiCad board)
At the start: 2 copper layers, 50 x 50 mm, 34 parts, among them J1 Conn_01x05, SW1 SW_DIP_x02, SW2 SW_Push, SW3 SW_Push, U1 CH340G, U2 CD4052B, U3 E18-MS1-PCB, U4 74LVC1G66, U5 74LVC1G66, U6 AP1117-33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

Commit message: add guide
Signed-off-by: SchumyHao <schumyhaojl@126.com>
Other:
- board text added: "Designed by smarthomefans"
- board text added: "TTY control 00 USB<=>ESP ZB<=>NC 01 USB<=>ZB ESP<=>NC 10 ESP<=>ZB USB<=>DBG 11 ESP<=>ZB USB<=>NC"
- board text added: "https://bbs.iobroker.cn"
- board text added: "z2m partner v01"
Changed lines of the file:
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@@
   (general
     (thickness 1.6)
-    (drawings 1)
+    (drawings 5)
     (tracks 511)
     (zones 0)
@@
     (39 F.Mask user hide)
     (40 Dwgs.User user)
-    (41 Cmts.User user hide)
+    (41 Cmts.User user)
     (42 Eco1.User user hide)
     (43 Eco2.User user hide)
@@
     (tags "capacitor handsolder")
     (attr smd)
-    (fp_text reference C7 (at 0.494 -1.43) (layer F.SilkS)
+    (fp_text reference C7 (at 2.526 0) (layer F.SilkS)
       (effects (font (size 1 1) (thickness 0.15)))
     )
@@
     (fp_line (start 2.45 -1.12) (end 2.45 1.12) (layer F.CrtYd) (width 0.05))
     (fp_line (start 2.45 1.12) (end -2.45 1.12) (layer F.CrtYd) (width 0.05))
-    (fp_text user %R (at 0 0 90) (layer F.Fab)
-      (effects (font (size 0.8 0.8) (thickness 0.12)))
+    (fp_text user PWR (at 1.8145 1.778 90) (layer F.SilkS)
+      (effects (font (size 0.8 0.8) (thickness 0.15)))
     )
     (pad 1 smd roundrect (at -1.4875 0 270) (size 1.425 1.75) (layers F.Cu F.Paste F.Mask) (roundrect_rratio 0.175439)
@@
     (fp_line (start 1.8 11.95) (end 1.8 -1.8) (layer F.CrtYd) (width 0.05))
     (fp_line (start 1.8 -1.8) (end -1.8 -1.8) (layer F.CrtYd) (width 0.05))
-    (fp_text user %R (at 0 5.08 45) (layer F.Fab)
-      (effects (font (size 1 1) (thickness 0.15)))
+    (fp_text user "G   D   C   R   V" (at -2.155261 5.028943 45) (layer F.SilkS)
+      (effects (font (size 0.8 0.8) (thickness 0.15)))
     )
     (pad 1 thru_hole rect (at 0 0 135) (size 1.7 1.7) (drill 1) (layers *.Cu *.Mask)
@@
       (effects (font (size 0.8 0.8) (thickness 0.12)))
     )
-    (fp_text user on (at 0.195 -1.395 135) (layer F.Fab)
+    (fp_text user on (at -1.885854 -2.604274 135) (layer F.SilkS)
       (effects (font (size 0.8 0.8) (thickness 0.12)))
     )
@@
     (fp_line (start 2.85 1.85) (end -2.85 1.85) (layer F.CrtYd) (width 0.05))
     (fp_line (start 2.85 -1.85) (end 2.85 1.85) (layer F.CrtYd) (width 0.05))
-    (fp_text user %R (at 0 0 45) (layer F.Fab)
-      (effects (font (size 0.6 0.6) (thickness 0.09)))
+    (fp_text user reset (at -0.71842 -2.514472 45) (layer F.SilkS)
+      (effects (font (size 0.8 0.8) (thickness 0.15)))
     )
     (fp_line (start 2.2 -1.58) (end 2.2 -1.7) (layer F.SilkS) (width 0.12))
@@
     (fp_line (start 2.2 0.57) (end 2.2 -0.57) (layer F.SilkS) (width 0.12))
     (fp_line (start 2.2 -1.58) (end 2.2 -1.7) (layer F.SilkS) (width 0.12))
-    (fp_text user %R (at 0 0 45) (layer F.Fab)
-      (effects (font (size 0.6 0.6) (thickness 0.09)))
+    (fp_text user flash (at -1.347038 -2.424669 45) (layer F.SilkS)
+      (effects (font (size 0.8 0.8) (thickness 0.15)))
     )
     (fp_line (start 2.85 -1.85) (end 2.85 1.85) (layer F.CrtYd) (width 0.05))
@@
     )
   )
+  (gr_text "TTY control\n00 USB<=>ESP\n    ZB<=>NC\n01 USB<=>ZB\n    ESP<=>NC\n10 ESP<=>ZB\n    USB<=>DBG\n11 ESP<=>ZB\n    USB<=>NC" (at 189.992 86.868) (layer B.SilkS)
+    (effects (font (size 1 1) (thickness 0.15)) (justify left mirror))
+  )
+  (gr_text https://bbs.iobroker.cn (at 185.166 125.222) (layer B.SilkS)
+    (effects (font (size 1 1) (thickness 0.15)) (justify mirror))
+  )
+  (gr_text "Designed by smarthomefans" (at 187.198 123.19) (layer B.SilkS)
+    (effects (font (size 1 1) (thickness 0.15)) (justify mirror))
+  )
+  (gr_text "z2m partner v01" (at 193.548 121.158) (layer B.SilkS)
+    (effects (font (size 1 1) (thickness 0.15)) (justify mirror))
+  )
   (gr_circle (center 184.55 102.87) (end 209.55 102.87) (layer Edge.Cuts) (width 0.12))
