File: project/z2m_partner.kicad_pcb (KiCad board)
At the start: 2 copper layers, 50 x 50 mm, 52 parts, among them J1 Conn_01x05, Q1 S8050, Q2 S8050, SW1 SW_DIP_x02, SW2 SW_Push, SW3 SW_Push, U1 CH340G, U2 CD4052B, U3 E18-MS1-PCB, U4 74LVC1G66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

Commit message: Update version to v02.1
Signed-off-by: SchumyHao <schumyhaojl@126.com>
Parts:
- D3, D6, D7, D8: value WS2812B -> SK6812_4020
- D4: renamed from D5; value WS2812B -> SK6812_4020
- D5: renamed from D4; value WS2812B -> SK6812_4020
- R13: value 0-NC -> 10k-NC
- R3, R4: value 10k-NC -> 10k
- R5, R9: value 12k -> 10k
- R6: value 0 -> 0-NC
- U1: value CH340G -> CH340C
- U3: value E18-MS1-PCB -> E18-MS1PA1-IPX
- U6: value AP1117-33 -> AMS1117-33
- Y1: value 12MHz -> 12MHz-NC
- turned R13 to 180 degrees
- turned R3 to 270 degrees
- turned R5 to 180 degrees
- turned R9 to 180 degrees
Connections:
- Q1 pad 1: /RTS -> Net-(Q1-Pad1)
- Q1 pad 2: Net-(Q1-Pad2) -> /RTS
- Q2 pad 1: /DTR -> Net-(Q2-Pad1)
- Q2 pad 2: Net-(Q2-Pad2) -> /DTR
- R13 pad 1: /SEL1 -> +3V3
- R13 pad 2: GND -> /SEL1
- R3 pad 1: +3V3 -> /SEL1
- R3 pad 2: /SEL1 -> GND
- R5 pad 2: Net-(Q1-Pad2) -> Net-(Q1-Pad1)
- R9 pad 2: Net-(Q2-Pad2) -> Net-(Q2-Pad1)
- U7 pad 14: /SEL0 -> /SEL1
- U7 pad 17: /SEL1 -> /SEL0
Routing:
- net GND: track 122.1 -> 112.1 mm, vias 179 -> 181
- net Net-(Q1-Pad1): track 0.00 -> 9.46 mm
- net Net-(Q1-Pad2): track 8.13 -> 0.00 mm
- net /SEL1: track 79.8 -> 71.7 mm, vias 2 -> 0
- net Net-(Q2-Pad1): track 0.00 -> 6.49 mm
- net +3V3: track 177.7 -> 183.4 mm, vias 6 -> 4
- net (no net): track 5.29 -> 0.00 mm
- net Net-(Q2-Pad2): track 4.49 -> 0.00 mm
- net /DTR: track 36.2 -> 39.8 mm
- net /SEL0: track 79.3 -> 82.5 mm, vias 4 -> 6
- net /ESP_IO0: track 24.2 -> 21.6 mm, vias 0 -> 2
- net /RTS: track 40.0 -> 41.0 mm
Other:
- board text added: "z2m partner v02.1"
- board text removed: "z2m partner v02"
