File: project/z2m_partner.sch (KiCad schematic (older format))
At the start: 32 parts, among them J1 Conn_01x05, SW1 SW_DIP_x02, SW2 SW_Push, SW3 SW_Push, U1 CH340G, U2 CD4052B, U3 E18-MS1-PCB, U4 74LVC1G66, U5 74LVC1G66, U6 AP1117-33, U7 ESP-WROOM-02, Y1 12MHz

Commit message: Update to v02
Signed-off-by: SchumyHao <schumyhaojl@126.com>
Parts:
- removed D1: LED, LED_SMD:LED_1206_3216Metric_Pad1.42x1.75mm_HandSolder, symbol Device:LED
- added C1, C10, C11, C12, C2, C8, C9: 100nF, Capacitor_SMD:C_0603_1608Metric_Pad1.05x0.95mm_HandSolder, symbol Device:C
- added D1: WS2812B, LED_SMD:LED_WS2812B_PLCC4_5.0x5.0mm_P3.2mm, symbol LED:WS2812B
- added D2: D, Diode_SMD:D_0603_1608Metric_Pad1.05x0.95mm_HandSolder, symbol Device:D
- added D3, D4, D5, D6, D7, D8: WS2812B, z2m_partner:SK6812_4020, symbol LED:WS2812B
- added Q1, Q2: S8050, Package_TO_SOT_SMD:TSOT-23, symbol Transistor_BJT:S8050
- added R13, R14: 0-NC, Resistor_SMD:R_0402_1005Metric, symbol Device:R_Small
- R3, R4: value 10k -> 10k-NC
- R5, R9: value 1k -> 12k; footprint Resistor_SMD:R_0805_2012Metric_Pad1.15x1.40mm_HandSolder -> Resistor_SMD:R_0603_1608Metric_Pad1.05x0.95mm_HandSolder
- R6, R8: footprint Resistor_SMD:R_0603_1608Metric_Pad1.05x0.95mm_HandSolder -> Resistor_SMD:R_0402_1005Metric
- Y1: footprint Crystal:Resonator_SMD_muRata_CSTxExxV-3Pin_3.0x1.1mm_HandSoldering -> Crystal:Resonator_SMD_muRata_CSTxExxV-3Pin_3.0x1.1mm
Connections:
- net +3V3: no longer R5.1
- net +5V: now also C10.2, C11.2, C12.2, C2.2, C8.2, C9.2, D2.2 (A), D3.1 (VDD), D4.1 (VDD), D5.1 (VDD), D6.1 (VDD), D7.1 (VDD), D8.1 (VDD); no longer R9.2
- net E18_P21: no longer U7.17 (IO16)
- net E18_P22: no longer R5.2
- net E18_RX: now also U2.12 (X0); no longer U2.14 (X1)
- net E18_TX: now also U2.1 (Y0); no longer U2.5 (Y1)
- net ESP_RST: now also Q1.3 (C)
- net ESP_RX: now also U2.14 (X1); no longer U2.12 (X0)
- net ESP_TX: now also U2.5 (Y1); no longer U2.1 (Y0)
- net GND: now also C1.1, C10.1, C11.1, C12.1, C2.1, C8.1, C9.1, D1.3 (VSS), D3.3 (VSS), D4.3 (VSS), D5.3 (VSS), D6.3 (VSS), D7.3 (VSS), D8.3 (VSS), R13.2, R14.2
- net SEL0: now also U7.14 (IO5), R14.1
- net SEL1: now also U7.17 (IO16), R13.1
- net DTR: now reaches U1.13 (~DTR)
- net DTR: now also R5.1, Q2.1 (E)
- net RTS: now reaches U1.14 (~RTS)
- net RTS: now also R9.1, Q1.1 (E)
- net LED: now reaches R12.1, U7.6 (IO15)
- net LED: now also D1.4 (DIN)
- net ESP_IO0: now reaches R11.2, SW3.1, U7.8 (IO0)
- net ESP_IO0: now also Q2.3 (C)
- new net: C1.2, D1.1 (VDD), D2.1 (K)
- new net: D1.2 (DOUT), D3.4 (DIN)
- new net: Q1.2 (B), R5.2
- new net: Q2.2 (B), R9.2
- new net: D7.2 (DOUT), D8.4 (DIN)
- new net: D6.2 (DOUT), D7.4 (DIN)
- new net: D5.2 (DOUT), D6.4 (DIN)
- new net: D3.2 (DOUT), D4.4 (DIN)
- new net: D4.2 (DOUT), D5.4 (DIN)
- no-connect marks 27 -> 26
Other:
- note added: "LED"
- note added: "V02"
- moved on the sheet: C5, C6, C7, F1, U6

Commit message: Update version to v02.1
Signed-off-by: SchumyHao <schumyhaojl@126.com>
Parts:
- removed Q1, Q2: S8050, Package_TO_SOT_SMD:TSOT-23, symbol Transistor_BJT:S8050
- added Q1, Q2: S8050, Package_TO_SOT_SMD:TSOT-23, symbol Device:Q_NPN_BEC
- D3, D4, D5, D6, D7, D8: value WS2812B -> SK6812_4020
- R13: renamed from R3; footprint Resistor_SMD:R_0603_1608Metric_Pad1.05x0.95mm_HandSolder -> Resistor_SMD:R_0402_1005Metric
- R3: renamed from R13; value 0-NC -> 10k; footprint Resistor_SMD:R_0402_1005Metric -> Resistor_SMD:R_0603_1608Metric_Pad1.05x0.95mm_HandSolder
- R4: value 10k-NC -> 10k
- R5, R9: value 12k -> 10k
- R6: value 0 -> 0-NC
- U1: value CH340G -> CH340C
- U3: value E18-MS1-PCB -> E18-MS1PA1-IPX
- U6: value AP1117-33 -> AMS1117-33
- Y1: value 12MHz -> 12MHz-NC
Connections:
- net DTR: now also Q2.2 (E)
- net ESP_IO0: now also Q2.3 (C)
- net ESP_RST: now also Q1.3 (C)
- net RTS: now also Q1.2 (E)
- net SEL0: now also U7.17 (IO16); no longer U7.14 (IO5)
- net SEL1: now also U7.14 (IO5); no longer U7.17 (IO16)
- net at R5.2: now also Q1.1 (B)
- net at R9.2: now also Q2.1 (B)
- no-connect marks 26 -> 25
Other:
- note added: "V02.1"
- note removed: "V02"
- moved on the sheet: C10, C11, C12, C2, C8, C9, D3, D4, D5, D6, D7, D8
